Commit message: Integrate Orbbec camera and visual calibration updates

File: src/car/urdf/car.urdf (robot description, URDF)
Before this commit: robot car, 21 links, 20 joints
Links:
- removed link camera_infra1_frame
- removed link camera_infra1_optical_frame
- added link base_root
- added link camera_bottom_screw_frame, mass 0.00583601107155577; collision mesh filename=package://orbbec_camera/meshes/astra2/camera_bottom_screw_f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; visual mesh filename=package://orbbec_camera/meshes/astra2/camera_bottom_screw_f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
- added link camera_ir_frame, mass 0.000608348661221201; collision mesh filename=package://orbbec_camera/meshes/astra2/camera_infra1_frame.S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; visual mesh filename=package://orbbec_camera/meshes/astra2/camera_infra1_frame.S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
- added link camera_ir_optical_frame, mass 0.000608348661221202; collision mesh filename=package://orbbec_camera/meshes/astra2/camera_infra1_optical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; visual mesh filename=package://orbbec_camera/meshes/astra2/camera_infra1_optical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
- link camera_color_frame: mass None -> 7.68929599151334E-05; geometry collision mesh filename=package://orbbec_camera/meshes/astra2/camera_colorl_frame.S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; visual mesh filename=package://orbbec_camera/meshes/astra2/camera_colorl_frame.S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
- link camera_color_optical_frame: mass None -> 7.68929599151334E-05; geometry collision mesh filename=package://orbbec_camera/meshes/astra2/camera_color_optical_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; visual mesh filename=package://orbbec_camera/meshes/astra2/camera_color_optical_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
- link camera_depth_frame: mass None -> 0.000608348661221201; geometry collision mesh filename=package://orbbec_camera/meshes/astra2/camera_depth_frame.STL; visual mesh filename=package://orbbec_camera/meshes/astra2/camera_depth_frame.STL
- link camera_depth_optical_frame: mass None -> 0.000608348661221202; geometry collision mesh filename=package://orbbec_camera/meshes/astra2/camera_depth_optical_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; visual mesh filename=package://orbbec_camera/meshes/astra2/camera_depth_optical_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
- link camera_link: mass 0.072 -> 0.0101524380243699; geometry collision mesh filename=package://orbbec_camera/meshes/astra2/base_link.STL; visual mesh filename=package://orbbec_camera/meshes/astra2/base_link.STL
Joints:
- removed joint camera_color_joint
- removed joint camera_color_optical_joint
- removed joint camera_depth_joint
- removed joint camera_depth_optical_joint
- removed joint camera_infra1_joint
- removed joint camera_infra1_optical_joint
- added joint base_root_joint: type fixed, parent base_root, child base_link, origin xyz=0 0 0 rpy=0 0 0
- added joint camera_bottom_screw_frame: type fixed, parent camera_link, child camera_bottom_screw_frame, origin xyz=-0.012323995999904 -0.0374999999985815 -0.0281503197112 rpy=0 0 0
- added joint camera_color_frame: type fixed, parent camera_depth_frame, child camera_color_frame, origin xyz=0.0025420000310987234 -0.01850000023841858 0 rpy=0 0 0
- added joint camera_color_optical_frame: type fixed, parent camera_color_frame, child camera_color_optical_frame, origin xyz=0 0 0 rpy=-1.5707963267949 0 -1.5707963267949
- added joint camera_depth_frame: type fixed, parent camera_link, child camera_depth_frame, origin xyz=0 0 0 rpy=0 0 0
- added joint camera_depth_optical_frame: type fixed, parent camera_depth_frame, child camera_depth_optical_frame, origin xyz=0 0 0 rpy=-1.5707963267949 0 -1.5707963267949
- added joint camera_ir_frame: type fixed, parent camera_depth_frame, child camera_ir_frame, origin xyz=0 0 0 rpy=0 0 0
- added joint camera_ir_optical_frame: type fixed, parent camera_ir_frame, child camera_ir_optical_frame, origin xyz=0 0 0 rpy=-1.5707963267949 0 -1.5707963267949
- joint camera_accel_joint: origin xyz=-0.01174 -0.00552 0.0051 rpy=0 0 0 -> xyz=0 0 0 rpy=0 0 0; parent camera_link -> camera_imu_frame
- joint camera_gyro_joint: origin xyz=-0.01174 -0.00552 0.0051 rpy=0 0 0 -> xyz=0 0 0 rpy=0 0 0; parent camera_link -> camera_imu_frame
- joint camera_imu_joint: origin xyz=-0.01174 -0.00552 0.0051 rpy=0 0 0 -> xyz=0 0 0 rpy=0 0 0
- joint camera_infra2_joint: origin xyz=0 -0.050 0 rpy=0 0 0 -> xyz=0 0 0 rpy=0 0 0; parent camera_link -> camera_ir_frame

Commit message: Update visual calibration mapping workflow

File: src/car/urdf/car.urdf (robot description, URDF)
Before this commit: robot car, 23 links, 22 joints
Links:
- removed link base_root
- added link imu_link, mass 0.041404; collision mesh filename=package://car/meshes/IMU.STL; visual mesh filename=package://car/meshes/IMU.STL
- added link left_ahead_swing_arm, mass 1.59994666091558; collision mesh filename=package://car/meshes/left_ahead_swing_arm.STL; visual mesh filename=package://car/meshes/left_ahead_swing_arm.STL
- added link left_back_swing_arm, mass 1.59994666091541; collision mesh filename=package://car/meshes/left_back_swing_arm.STL; visual mesh filename=package://car/meshes/left_back_swing_arm.STL
- added link right_ahead_swing_arm, mass 1.59994666091772; collision mesh filename=package://car/meshes/right_ahead_swing_arm.STL; visual mesh filename=package://car/meshes/right_ahead_swing_arm.STL
- added link right_back_swing_arm, mass 1.59994666091541; collision mesh filename=package://car/meshes/right_back_swing_arm.STL; visual mesh filename=package://car/meshes/right_back_swing_arm.STL
- link base_link: mass 28.419 -> 14.5049759407965
- link camera_bottom_screw_frame: mass 0.00583601107155577 -> None; geometry 
- link camera_color_frame: mass 7.68929599151334E-05 -> None; geometry 
- link camera_color_optical_frame: mass 7.68929599151334E-05 -> None; geometry 
- link camera_depth_frame: mass 0.000608348661221201 -> None; geometry 
- link camera_depth_optical_frame: mass 0.000608348661221202 -> None; geometry 
- link camera_ir_frame: mass 0.000608348661221201 -> None; geometry 
- link camera_ir_optical_frame: mass 0.000608348661221202 -> None; geometry 
- link camera_link: mass 0.0101524380243699 -> 0.22447; geometry collision mesh filename=package://car/meshes/Astra2.STL; visual mesh filename=package://car/meshes/Astra2.STL
- link left_ahead_wheel: mass 0.048775 -> 0.0766649138440825; geometry collision mesh filename=package://car/meshes/wheel3.STL; visual mesh filename=package://car/meshes/wheel3.STL
- link left_back_wheel: mass 0.048775 -> 0.0766649138440825; geometry collision mesh filename=package://car/meshes/wheel1.STL; visual mesh filename=package://car/meshes/wheel1.STL
- link lidar: mass 0.74292 -> 0.1808; geometry collision mesh filename=package://car/meshes/rplidar_a3.STL; visual mesh filename=package://car/meshes/rplidar_a3.STL
- link right_ahead_wheel: mass 0.048775 -> 0.0766649138440825; geometry collision mesh filename=package://car/meshes/wheel4.STL; visual mesh filename=package://car/meshes/wheel4.STL
- link right_back_wheel: mass 0.048775 -> 0.0766649138440825; geometry collision mesh filename=package://car/meshes/wheel2.STL; visual mesh filename=package://car/meshes/wheel2.STL
Joints:
- removed joint base_root_joint
- added joint imu_joint: type fixed, parent base_link, child imu_link, origin xyz=0 -0.095 0.261 rpy=1.5708 0 3.1416, axis 0 0 0
- added joint left_ahead_swing_arm_joint: type continuous, parent base_link, child left_ahead_swing_arm, origin xyz=0.251499999999997 0.267109528305623 0.064993016915769 rpy=1.5707963267949 0 -3.14159265358979, axis 1 0 0
- added joint left_back_swing_arm_joint: type continuous, parent base_link, child left_back_swing_arm, origin xyz=-0.2515 0.267109528305508 0.0649930169157672 rpy=1.5707963267949 0 3.14159265358979, axis -1 0 0
- added joint right_ahead_swing_arm_joint: type continuous, parent base_link, child right_ahead_swing_arm, origin xyz=0.251499999999997 -0.266889266941522 0.0661273337114879 rpy=1.5707963267949 0 -3.14159265358979, axis 1 0 0
- added joint right_back_swing_arm_joint: type continuous, parent base_link, child right_back_swing_arm, origin xyz=-0.249000000000455 -0.266889266928036 0.0661273337114438 rpy=1.5707963267949 0 3.14159265358979, axis -1 0 0
- joint camera_joint: axis (none) -> 0 0 0; origin xyz=0.2549 -0.0037612 0.22883 rpy=0 0 0 -> xyz=0 -0.308 0.228 rpy=1.5708 0 3.1416
- joint left_ahead_wheel_joint: axis 0 1 0 -> 1 0 0; origin xyz=0.156 0.219 0 rpy=0 0 0 -> xyz=0.215999999999997 0.174999278050727 0.013188559598079 rpy=1.5707963267949 0 -3.14159265358979
- joint left_back_wheel_joint: axis 0 1 0 -> -1 0 0; origin xyz=-0.156 0.219 0 rpy=0 0 0 -> xyz=-0.216000000000004 0.174999278050617 0.0131885595980792 rpy=1.5707963267949 0 3.14159265358979
- joint lidar_joint: origin xyz=0.1555 -0.0010002 0.3007 rpy=0 0 0 -> xyz=0.00083897 -0.18046 0.38393 rpy=0.0217036732051 -0.0032179 3.1415
- joint right_ahead_wheel_joint: axis 0 1 0 -> 1 0 0; origin xyz=0.156 -0.219 0 rpy=0 0 0 -> xyz=0.215999999999997 -0.172799937280656 0.0139273524474186 rpy=1.5707963267949 0 -3.14159265358979
- joint right_back_wheel_joint: axis 0 1 0 -> -1 0 0; origin xyz=-0.156 -0.219 0 rpy=0 0 0 -> xyz=-0.216000000000004 -0.174999932317364 0.0139320256626821 rpy=1.5707963267949 0 3.14159265358979
