Commit message: Update rebo24 simulation config and docs

File: src/rebo24/urdf/rebo24.urdf (robot description, URDF)
Before this commit: robot rebo24, 23 links, 22 joints
Links:
- removed link camera
- removed link imu
- added link imu_link, mass 0.105365739619058; collision mesh filename=package://rebo24/meshes/imu_link.STL; visual mesh filename=package://rebo24/meshes/imu_link.STL
- link base_link: mass 43.083 -> 43.0826866003702
- link camera_link: mass 1e-06 -> 0.048201398677882; geometry collision mesh filename=package://rebo24/meshes/camera_link.STL; visual mesh filename=package://rebo24/meshes/camera_link.STL
- link left_ahead_wheel: mass 0.076906 -> 0.0769061881598781
- link right_ahead_wheel: mass 0.076906 -> 0.0769061881598782
- link right_back_wheel: mass 0.076906 -> 0.0769061881598782
Joints:
- removed joint camera_visual_joint
- joint camera_accel_joint: axis 0 0 0 -> (none); origin xyz=-0.0955 -0.00048109 -0.06477 rpy=0 0 0 -> xyz=-0.01174 -0.00552 0.0051 rpy=0 0 0
- joint camera_accel_optical_joint: axis 0 0 0 -> (none)
- joint camera_color_joint: axis 0 0 0 -> (none)
- joint camera_color_optical_joint: axis 0 0 0 -> (none)
- joint camera_depth_joint: axis 0 0 0 -> (none)
- joint camera_depth_optical_joint: axis 0 0 0 -> (none)
- joint camera_gyro_joint: axis 0 0 0 -> (none); origin xyz=-0.0955 -0.00048109 -0.06477 rpy=0 0 0 -> xyz=-0.01174 -0.00552 0.0051 rpy=0 0 0
- joint camera_gyro_optical_joint: axis 0 0 0 -> (none)
- joint camera_imu_joint: axis 0 0 0 -> (none); origin xyz=-0.0955 -0.00048109 -0.06477 rpy=0 0 0 -> xyz=-0.01174 -0.00552 0.0051 rpy=0 0 0
- joint camera_imu_optical_joint: axis 0 0 0 -> (none)
- joint camera_infra1_joint: axis 0 0 0 -> (none)
- joint camera_infra1_optical_joint: axis 0 0 0 -> (none)
- joint camera_infra2_joint: axis 0 0 0 -> (none)
- joint camera_infra2_optical_joint: axis 0 0 0 -> (none)
- joint camera_joint: origin xyz=0.2655 -0.00051911 0.24872 rpy=0 0 0 -> xyz=0.265499999999739 -0.000519114270499249 0.248720793604667 rpy=0 0 0
- joint imu_joint: child imu -> imu_link; origin xyz=0 0 0 rpy=0 0 0 -> xyz=0.169999999947848 -0.00100019470600629 0.183950000000706 rpy=0 0 0; parent camera_imu_frame -> base_link
- joint left_ahead_wheel_joint: origin xyz=0.1415 0.233 0 rpy=0 0 0 -> xyz=0.141499999999909 0.233000195879141 0 rpy=0 0 0
- joint left_back_wheel_joint: origin xyz=-0.1415 0.233 0 rpy=0 0 0 -> xyz=-0.141500000000089 0.233000195879139 0 rpy=0 0 0
- joint lidar_joint: origin xyz=0.17 -0.0010002 0.3057 rpy=0 0 0 -> xyz=0.169999999999687 -0.00100019587911868 0.305700000000706 rpy=0 0 0
- joint right_back_wheel_joint: origin xyz=-0.1415 -0.233 0 rpy=0 0 0 -> xyz=-0.14149999999997 -0.233000195879138 0 rpy=0 0 0
